File: hardware/solenoid_1ch.sch (EAGLE design)
At the start: 18 parts, among them U2 AP2204R

Commit message: Added protection diodes
Parts:
- added D1: (no value), microbuilder:DIODESOD-123
Connections:
- net N$12: now also D1.A
- net VDD: now also D1.C
Changed lines of the file:
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@@
 <part name="GND13" library="SparkFun-Aesthetics" deviceset="GND2" device=""/>
 <part name="R8" library="SparkFun-Passives" deviceset="RESISTOR" device="0805-RES" value="100"/>
+<part name="D1" library="microbuilder" deviceset="DIODE" device="SOD-123"/>
 </parts>
 <sheets>
@@
 <instance part="GND13" gate="G$1" x="91.44" y="121.92"/>
 <instance part="R8" gate="G$1" x="78.74" y="132.08" rot="R270"/>
+<instance part="D1" gate="G$1" x="132.08" y="185.42" rot="R90"/>
 </instances>
 <busses>
@@
 <segment>
 <pinref part="SUPPLY12" gate="VDD" pin="VDD"/>
-<wire x1="139.7" y1="190.5" x2="139.7" y2="185.42" width="0.1524" layer="91"/>
+<wire x1="139.7" y1="190.5" x2="139.7" y2="187.96" width="0.1524" layer="91"/>
 <pinref part="OUT-R" gate="G$1" pin="1"/>
+<wire x1="139.7" y1="187.96" x2="139.7" y2="185.42" width="0.1524" layer="91"/>
 <wire x1="139.7" y1="185.42" x2="142.24" y2="185.42" width="0.1524" layer="91"/>
+<pinref part="D1" gate="G$1" pin="C"/>
+<wire x1="132.08" y1="187.96" x2="139.7" y2="187.96" width="0.1524" layer="91"/>
 </segment>
 <segment>
@@
 <pinref part="$T3" gate="G$1" pin="D"/>
 <wire x1="137.16" y1="182.88" x2="137.16" y2="172.72" width="0.1524" layer="91"/>
-</segment>
-</net>
+<pinref part="D1" gate="G$1" pin="A"/>
+<wire x1="132.08" y1="182.88" x2="137.16" y2="182.88" width="0.1524" layer="91"/>
+</segment>
+</net>
